File: pcb/Vario 0.1 Ultra Mini.brd (EAGLE design)
At the start: 17.1 x 22.1 mm, 28 parts

Commit message: doc
Parts:
- MS5611: value (none) -> MS5607PACKAGEDNORMAL
Connections:
- net GND: now also MS5611.3, MS5611.4; no longer MS5611.P$3, MS5611.P$4
- net SCL: now also MS5611.8; no longer MS5611.P$8
- net SDA: now also MS5611.7; no longer MS5611.P$7
- net SYS_LOAD: now also MS5611.1, MS5611.2; no longer MS5611.P$1, MS5611.P$2
