File: pcb/Vario 0.1 Ultra Mini.sch (EAGLE design)
At the start: 28 parts

Commit message: doc
Parts:
- MS5611: value MS5607PACKAGED -> MS5607PACKAGEDNORMAL; device measurement_specialties:MS5607PACKAGED -> measurement_specialties:MS5607PACKAGEDNORMAL
